File: cm4-gpio.kicad_sch (KiCad schematic)
At the start: 5 parts, among them J2 DF40C-100DP-0.4V_51_

Commit message: cleanup
Parts:
- removed J2: DF40C-100DP-0.4V_51_, ulx5m-gs:HRS_DF40C-100DP-0.4V_51_, symbol DF40C-100DP-0.4V_51_:DF40C-100DP-0.4V_51_
