File: cm4-hsio.kicad_sch (KiCad schematic)
At the start: 3 parts, among them J1 DF40C-100DP-0.4V_51_

Commit message: cleanup
Parts:
- removed J1: DF40C-100DP-0.4V_51_, ulx5m-gs:HRS_DF40C-100DP-0.4V_51_, symbol DF40C-100DP-0.4V_51_:DF40C-100DP-0.4V_51_
