File: ethernet.kicad_sch (KiCad schematic)
At the start: 92 parts, among them J5 USB_C_Receptacle, Q1 BSS138, Q2 BSS138, U14 KSZ9031RNXCA, U4 GateMate-CCGM1A1, X1 ECS-2520MV-250-xx

Commit message: cleanup
Connections:
- net LED1#: now reaches U4.G16 (IO_EA_A8)
- net PEDET: now reaches U4.G17 (IO_EA_B7)
- net ID_SC renamed PEWAKE#
- net ID_SD renamed CLKREQ#
- net PWR_BTN renamed SUSCLK
- net SCL0 renamed PERST#
- net SDA0 renamed DEVSLP
Changed lines of the file:
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@@
 	)
 	(bus_entry
-		(at 40.64 74.93)
-		(size -2.54 2.54)
-		(stroke
-			(width 0)
-			(type default)
-		)
-	)
-	(bus_entry
 		(at 132.08 189.23)
 		(size -2.54 2.54)
@@
 	)
 	(bus_entry
-		(at 40.64 72.39)
-		(size -2.54 2.54)
-		(stroke
-			(width 0)
-			(type default)
-		)
-	)
-	(bus_entry
 		(at 248.92 104.14)
 		(size 2.54 2.54)
@@
 	)
 	(bus_entry
-		(at 40.64 80.01)
-		(size -2.54 2.54)
-		(stroke
-			(width 0)
-			(type default)
-		)
-	)
-	(bus_entry
 		(at 248.92 101.6)
 		(size 2.54 2.54)
@@
 	)
 	(bus_entry
-		(at 40.64 77.47)
-		(size -2.54 2.54)
-		(stroke
-			(width 0)
-			(type default)
-		)
-	)
-	(bus_entry
 		(at 248.92 116.84)
 		(size 2.54 2.54)
@@
 	(wire
 		(pts
-			(xy 40.64 72.39) (xy 55.88 72.39)
-		)
-		(stroke
-			(width 0)
-			(type default)
-		)
-	)
-	(wire
-		(pts
 			(xy 167.64 20.32) (xy 167.64 21.59)
 		)
@@
 	(wire
 		(pts
+			(xy 50.8 87.63) (xy 55.88 87.63)
+		)
+		(stroke
+			(width 0)
+			(type default)
+		)
+	)
+	(wire
+		(pts
 			(xy 203.2 63.5) (xy 205.74 63.5)
 		)
@@
 	(wire
 		(pts
+			(xy 52.07 74.93) (xy 55.88 74.93)
+		)
+		(stroke
+			(width 0)
+			(type default)
+		)
+	)
+	(wire
+		(pts
 			(xy 91.44 46.99) (xy 115.57 46.99)
 		)
@@
 	(wire
 		(pts
-			(xy 40.64 80.01) (xy 55.88 80.01)
+			(xy 302.26 73.66) (xy 302.26 76.2)
 		)
 		(stroke
@@
 	(wire
 		(pts
-			(xy 302.26 73.66) (xy 302.26 76.2)
+			(xy 232.41 207.01) (xy 238.76 207.01)
 		)
 		(stroke
@@
 	(wire
 		(pts
-			(xy 232.41 207.01) (xy 238.76 207.01)
+			(xy 74.93 121.92) (xy 81.28 121.92)
 		)
 		(stroke
@@
 	(wire
 		(pts
-			(xy 74.93 121.92) (xy 81.28 121.92)
+			(xy 27.94 129.54) (xy 34.29 129.54)
 		)
 		(stroke
@@
 	(wire
 		(pts
-			(xy 27.94 129.54) (xy 34.29 129.54)
+			(xy 52.07 77.47) (xy 55.88 77.47)
 		)
 		(stroke
@@
 	(wire
 		(pts
-			(xy 40.64 77.47) (xy 55.88 77.47)
-		)
-		(stroke
-			(width 0)
-			(type default)
-		)
-	)
-	(wire
-		(pts
 			(xy 27.94 121.92) (xy 27.94 124.46)
 		)
@@
 		)
 	)
-	(bus
-		(pts
-			(xy 38.1 74.93) (xy 38.1 77.47)
-		)
-		(stroke
-			(width 0)
-			(type default)
-		)
-	)
 	(wire
 		(pts
@@
 	(wire
 		(pts
-			(xy 55.88 74.93) (xy 40.64 74.93)
-		)
-		(stroke
-			(width 0)
-			(type default)
-		)
-	)
-	(wire
-		(pts
 			(xy 284.48 91.44) (xy 284.48 92.71)
 		)
@@
 	(wire
 		(pts
+			(xy 52.07 72.39) (xy 55.88 72.39)
+		)
+		(stroke
+			(width 0)
+			(type default)
+		)
+	)
+	(wire
+		(pts
 			(xy 85.09 185.42) (xy 88.9 185.42)
 		)
@@
 		)
 	)
-	(bus
-		(pts
-			(xy 38.1 80.01) (xy 38.1 82.55)
-		)
-		(stroke
-			(width 0)
-			(type default)
-		)
-	)
 	(wire
 		(pts
@@
 	(wire
 		(pts
+			(xy 50.8 85.09) (xy 55.88 85.09)
+		)
+		(stroke
+			(width 0)
+			(type default)
+		)
+	)
+	(wire
+		(pts
 			(xy 111.76 69.85) (xy 127 69.85)
 		)
@@
 		)
 	)
-	(bus
-		(pts
-			(xy 38.1 77.47) (xy 38.1 80.01)
-		)
-		(stroke
-			(width 0)
-			(type default)
-		)
-	)
 	(wire
 		(pts
@@
 	(wire
 		(pts
+			(xy 52.07 80.01) (xy 55.88 80.01)
+		)
+		(stroke
+			(width 0)
+			(type default)
+		)
+	)
+	(wire
+		(pts
 			(xy 96.52 34.29) (xy 106.68 34.29)
 		)
@@
 		)
 	)
-	(bus
-		(pts
-			(xy 38.1 82.55) (xy 33.02 82.55)
-		)
-		(stroke
-			(width 0)
-			(type default)
-		)
-	)
 	(wire
 		(pts
@@
 		)
 	)
-	(label "ID_SC"
-		(at 50.8 80.01 180)
-		(effects
-			(font
-				(size 1.27 1.27)
-			)
-			(justify right bottom)
-		)
-	)
 	(label "USB_P"
 		(at 134.62 189.23 0)
@@
 		)
 	)
-	(label "ID_SD"
-		(at 50.8 77.47 180)
-		(effects
-			(font
-				(size 1.25 1.25)
-			)
-			(justify right bottom)
-		)
-	)
 	(label "RGMII_RX_DV"
 		(at 137.16 106.68 0)
@@
 		)
 	)
-	(label "SCL0"
-		(at 45.72 74.93 0)
-		(effects
-			(font
-				(size 1.27 1.27)
-			)
-			(justify left bottom)
-		)
-	)
 	(label "RGMII_TXE"
 		(at 100.33 54.61 180)
@@
 		)
 	)
-	(label "SDA0"
-		(at 45.72 72.39 0)
-		(effects
-			(font
-				(size 1.27 1.27)
-			)
-			(justify left bottom)
-		)
-	)
 	(label "FPD1-"
 		(at 59.69 193.04 0)
@@
 		)
 	)
-	(global_label "PWR_BTN"
-		(shape input)
-		(at 50.8 82.55 180)
-		(fields_autoplaced yes)
-		(effects
-			(font
-				(size 1.254 1.254)
-			)
-			(justify right)
-		)
-		(property "Intersheetrefs" "${INTERSHEET_REFS}"
-			(at 39.4328 82.55 0)
-			(effects
-				(font
-					(size 1.27 1.27)
-				)
-				(justify right)
-				(hide yes)
-			)
-		)
-	)
 	(global_label "VDD_CLK"
 		(shape output)
@@
 		)
 	)
+	(hierarchical_label "LED1#"
+		(shape output)
+		(at 50.8 87.63 180)
+		(effects
+			(font
+				(size 1.27 1.27)
+			)
+			(justify right)
+		)
+	)
 	(hierarchical_label "USB_CC1"
 		(shape passive)
@@
 		)
 	)
+	(hierarchical_label "DEVSLP"
+		(shape input)
+		(at 52.07 72.39 180)
+		(effects
+			(font
+				(size 1.27 1.27)
+			)
+			(justify right)
+		)
+	)
+	(hierarchical_label "SUSCLK"
+		(shape input)
+		(at 50.8 82.55 180)
+		(effects
+			(font
+				(size 1.27 1.27)
+			)
+			(justify right)
+		)
+	)
+	(hierarchical_label "CLKREQ#"
+		(shape bidirectional)
+		(at 52.07 77.47 180)
+		(effects
+			(font
+				(size 1.27 1.27)
+			)
+			(justify right)
+		)
+	)
 	(hierarchical_label "{ETH}"
 		(shape bidirectional)
@@
 		)
 	)
+	(hierarchical_label "PEDET"
+		(shape output)
+		(at 50.8 85.09 180)
+		(effects
+			(font
+				(size 1.27 1.27)
+			)
+			(justify right)
+		)
+	)
 	(hierarchical_label "{USB}"
 		(shape bidirectional)
@@
 		)
 	)
-	(hierarchical_label "{ETH}"
+	(hierarchical_label "PERST#"
+		(shape input)
+		(at 52.07 74.93 180)
+		(effects
+			(font
+				(size 1.27 1.27)
+			)
+			(justify right)
+		)
+	)
+	(hierarchical_label "PEWAKE#"
 		(shape bidirectional)
-		(at 281.94 129.54 180)
+		(at 52.07 80.01 180)
 		(effects
 			(font
@@
 		)
 	)
-	(hierarchical_label "{I2C}"
+	(hierarchical_label "{ETH}"
 		(shape bidirectional)
-		(at 33.02 82.55 180)
+		(at 281.94 129.54 180)
 		(effects
 			(font
