File: ethernet.kicad_sch (KiCad schematic)
At the start: 92 parts, among them J5 USB_C_Receptacle, Q1 BSS138, Q2 BSS138, U14 KSZ9031RNXCA, U4 GateMate-CCGM1A1, X1 ECS-2520MV-250-xx

Commit message: Version 1.0
Parts:
- removed C104, C105, C109, C114: 10u, Capacitor_SMD:C_0402_1005Metric, symbol Device:C_Small
- removed C106, C107, C108, C112, C116, C117, C118: 100n, Capacitor_SMD:C_0402_1005Metric, symbol Device:C_Small
- removed C110, C111, C113, C119: 10n, Capacitor_SMD:C_0402_1005Metric, symbol Device:C_Small
- removed C115: 4u7, Capacitor_SMD:C_0402_1005Metric, symbol Device:C_Small
- removed FB1, FB2, FB3: BLM18PG121SN1D, Inductor_SMD:L_0603_1608Metric, symbol Device:FerriteBead_Small
- removed Q1, Q2: BSS138, Package_TO_SOT_SMD:SOT-523, symbol Transistor_FET:BSS138
- removed R100, R101, R102, R104, R89, R90, R91, R92, R93, R94, R97, R98, R99: 27R, Resistor_SMD:R_0402_1005Metric, symbol Device:R_Small
- removed R103: 12k1, Resistor_SMD:R_0402_1005Metric, symbol Device:R_Small
- removed R66, R67, R70, R71, R72, R73, R78, R79, R84, R85, R96: 4k7, Resistor_SMD:R_0402_1005Metric, symbol Device:R_Small
- removed R68, R69, R74, R75, R76, R77, R80, R81, R82, R83: dnp, Resistor_SMD:R_0402_1005Metric, symbol Device:R_Small
- removed U14: KSZ9031RNXCA, Package_DFN_QFN:QFN-48-1EP_7x7mm_P0.5mm_EP5.15x5.15mm, symbol Interface_Ethernet:KSZ9031RNXCA
- removed X1: ECS-2520MV-250-xx, Oscillator:Oscillator_SMD_ECS_2520MV-xxx-xx-4Pin_2.5x2.0mm, symbol Oscillator:ECS-2520MV-xxx-xx
Connections:
- net CLKREQ#: no longer names the net of U4.H16 (IO_EA_A6)
- net DEVSLP: no longer names the net of U4.J16 (IO_EA_A5)
- net ETH_CLK: no longer names the net of U4.E16 (IO_EB_A3)
- net LED1#: no longer names the net of U4.G16 (IO_EA_A8)
- net PEDET: no longer names the net of U4.G17 (IO_EA_B7)
- net PERST#: no longer names the net of U4.J15 (IO_EA_B5)
- net PEWAKE#: no longer names the net of U4.H15 (IO_EA_B6)
- net RGMII_INT_N: no longer names the net of U4.C15 (IO_EB_B7)
- net RGMII_MDC: no longer names the net of U4.C16 (IO_EB_B6)
- net RGMII_MDIO: no longer names the net of U4.D16 (IO_EB_A6)
- net RGMII_REFCLK: no longer names the net of U4.A15 (IO_EB_B8)
- net RGMII_RST_N: no longer names the net of U4.E15 (IO_EB_B3)
- net RGMII_RXD0: no longer names the net of U4.F18 (IO_EB_A0)
- net RGMII_RXD1: no longer names the net of U4.F17 (IO_EB_B0)
- net RGMII_RXD2: no longer names the net of U4.F16 (IO_EB_A1)
- net RGMII_RXD3: no longer names the net of U4.F15 (IO_EB_B1)
- net RGMII_RX_CLK: no longer names the net of U4.D15 (IO_EB_A7)
- net RGMII_RX_DV: no longer names the net of U4.B15 (IO_EB_A8)
- net RGMII_TX0: no longer names the net of U4.A17 (IO_EB_B5)
- net RGMII_TX1: no longer names the net of U4.B17 (IO_EB_A5)
- net RGMII_TX2: no longer names the net of U4.C17 (IO_EB_B4)
- net RGMII_TX3: no longer names the net of U4.C18 (IO_EB_A4)
- net RGMII_TXE: no longer names the net of U4.D18 (IO_EB_A2)
- net RGMII_TX_CK: no longer names the net of U4.D17 (IO_EB_B2)
- net SUSCLK: no longer names the net of U4.G18 (IO_EA_A7)
- no-connect marks 2 -> 0
Other:
- note removed: "CLK125_EN: 0: disable / 1: enable"
- note removed: "LED_MODE: 0: tri-color / 1: single-led"
- note removed: "MODE0"
- note removed: "MODE1"
- note removed: "MODE2"
- note removed: "MODE3"
- note removed: "PHYAD0"
- note removed: "PHYAD1"
- note removed: "PHYAD2"
- note removed: "PME_N2: 0: WOL events / 1: INT events"
- note removed: "Strap Options"
- note removed: "Use EB-A3 as clock source Or use EB-A3 as input and place X1, C118, R104"
