File: lvds.kicad_sch (KiCad schematic)
At the start: 52 parts, among them U4 GateMate-CCGM1A1, Y1 ASE2-25.000MHZ-L-C-T

Commit message: cleanup
Parts:
- removed C59, C60, C61, C62, C63, C64, C65, C66: 220n, Capacitor_SMD:C_0402_1005Metric, symbol Device:C_Small
