File: power.kicad_sch (KiCad schematic)
At the start: 87 parts, among them J3 Vcore_sel, U1 TLV62569DBV, U2 TLV62569DBV, U3 MPM3833CGRH-Z, U4 GateMate-CCGM1A1, U5 TLV62569DBV

Commit message: cleanup
Parts:
- removed C3: 4u7, Capacitor_SMD:C_0402_1005Metric, symbol Device:C_Small
- removed C7: 10u, Capacitor_SMD:C_0402_1005Metric, symbol Device:C_Small
- removed C9: 1u, Capacitor_SMD:C_0402_1005Metric, symbol Device:C_Small
- removed L2: DFE322512F-2R2M=P2, Inductor_SMD:L_1008_2520Metric, symbol Device:L_Small
- removed R11: 0R, Resistor_SMD:R_0603_1608Metric, symbol Device:R_Small
- removed R5: 100k, Resistor_SMD:R_0402_1005Metric, symbol Device:R_Small
- removed R6: 22k, Resistor_SMD:R_0402_1005Metric, symbol Device:R_Small
- removed TP2: 3V3, TestPoint:TestPoint_Pad_D1.0mm, symbol Connector:TestPoint
- removed U2: TLV62569DBV, Package_TO_SOT_SMD:SOT-23-5, symbol Regulator_Switching:TLV62569DBV
Other:
- note added: "Needs to be 3.3V input"
- note removed: "0.6*(1+(100/22))=3.327"
