File: config.kicad_sch (KiCad schematic)
At the start: 41 parts, among them J4 JTAG, SW1 219-2MST, U4 GateMate-CCGM1A1, U6 74LVC1G04GM,115, U7 74LVC2G00HK3-7, U8 74LVC2G00HK3-7, U9 AT25QL321-MBUE-T

Commit message: Version 1.0
Parts:
- J4: now fitted; now in the parts list
- R147, R148, R149, R150: now not fitted; now left out of the parts list
Changed lines of the file:
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@@
 		(unit 1)
 		(exclude_from_sim no)
-		(in_bom yes)
-		(on_board yes)
-		(dnp no)
+		(in_bom no)
+		(on_board no)
+		(dnp yes)
 		(property "Reference" "R148"
 			(at 46.228 104.14 90)
@@
 		(unit 1)
 		(exclude_from_sim no)
-		(in_bom yes)
-		(on_board yes)
-		(dnp no)
+		(in_bom no)
+		(on_board no)
+		(dnp yes)
 		(property "Reference" "R149"
 			(at 46.228 106.68 90)
@@
 		(unit 1)
 		(exclude_from_sim no)
-		(in_bom no)
+		(in_bom yes)
 		(on_board yes)
-		(dnp yes)
+		(dnp no)
 		(fields_autoplaced yes)
 		(property "Reference" "J4"
@@
 			)
 		)
+		(property "LCSC" ""
+			(at 256.54 127 0)
+			(effects
+				(font
+					(size 1.27 1.27)
+				)
+				(hide yes)
+			)
+		)
 		(pin "1"
 		)
@@
 		(unit 1)
 		(exclude_from_sim no)
-		(in_bom yes)
-		(on_board yes)
-		(dnp no)
+		(in_bom no)
+		(on_board no)
+		(dnp yes)
 		(property "Reference" "R147"
 			(at 46.228 101.854 90)
@@
 		(unit 1)
 		(exclude_from_sim no)
-		(in_bom yes)
-		(on_board yes)
-		(dnp no)
+		(in_bom no)
+		(on_board no)
+		(dnp yes)
 		(property "Reference" "R150"
 			(at 46.228 109.474 90)
