File: config.kicad_sch (KiCad schematic)
At the start: 41 parts, among them J4 JTAG, SW1 219-2MST, U4 GateMate-CCGM1A1, U6 74LVC1G04GM,115, U7 74LVC2G00HK3-7, U8 74LVC2G00HK3-7, U9 AT25QL321-MBUE-T

Commit message: Switching to 6L board - routing - adding schemaitcs
Parts:
- removed JP1: POR_EN, Jumper:SolderJumper-2_P1.3mm_Open_RoundedPad1.0x1.5mm, symbol Jumper:SolderJumper_2_Open
- added J101: JTAG_EXT, Connector_PinHeader_1.27mm:PinHeader_1x04_P1.27mm_Vertical, symbol Connector:Conn_01x04_Pin
- added J102: 3V3_PSU, Connector_PinHeader_1.27mm:PinHeader_1x02_P1.27mm_Vertical, symbol Connector:Conn_01x02_Pin
- added R66: dnp, Resistor_SMD:R_0402_1005Metric, symbol Device:R_Small
Connections:
- net +1V8: now also R66.1
- net GND: now also J102.2 (Pin_2)
- net JTAG_POR: now also R66.2
- net at J4.4 (Pin_4), R43.2: now also J101.4 (Pin_4)
- net at J4.1 (Pin_1), R40.2: now also J101.1 (Pin_1)
- net at J4.2 (Pin_2), R41.2: now also J101.2 (Pin_2)
- net at J4.3 (Pin_3), R42.2: now also J101.3 (Pin_3)
- new net +3V3: J102.1 (Pin_1)
Other:
- note added: "POR_EN"
- moved on the sheet: R40, R41, R42, R43
