File: gpio.kicad_sch (KiCad schematic)
At the start: 11 parts, among them U4 GateMate-CCGM1A1

Commit message: Version 1.0
Connections:
- net GPIO12 renamed PEDET
- net GPIO18 renamed LED1#
- net GPIO23 renamed DEVSLP
- net GPIO24 renamed PERST#
- net GPIO25 renamed CLKREQ#
- net GPIO7 renamed SUSCLK
- net GPIO8 renamed PEWAKE#
Changed lines of the file:
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@@
+	(wire
+		(pts
+			(xy 218.44 85.09) (xy 223.52 85.09)
+		)
+		(stroke
+			(width 0)
+			(type default)
+		)
+	)
 	(wire
 		(pts
@@
 		)
 	)
+	(wire
+		(pts
+			(xy 218.44 80.01) (xy 223.52 80.01)
+		)
+		(stroke
+			(width 0)
+			(type default)
+		)
+	)
 	(bus
 		(pts
@@
 	(wire
 		(pts
+			(xy 219.71 69.85) (xy 223.52 69.85)
+		)
+		(stroke
+			(width 0)
+			(type default)
+		)
+	)
+	(wire
+		(pts
 			(xy 175.26 38.1) (xy 175.26 39.37)
 		)
@@
 	(wire
 		(pts
+			(xy 219.71 72.39) (xy 223.52 72.39)
+		)
+		(stroke
+			(width 0)
+			(type default)
+		)
+	)
+	(wire
+		(pts
 			(xy 170.18 60.96) (xy 180.34 60.96)
 		)
@@
 	(wire
 		(pts
+			(xy 219.71 77.47) (xy 223.52 77.47)
+		)
+		(stroke
+			(width 0)
+			(type default)
+		)
+	)
+	(wire
+		(pts
 			(xy 170.18 55.88) (xy 180.34 55.88)
 		)
@@
 		)
 	)
+	(wire
+		(pts
+			(xy 218.44 82.55) (xy 223.52 82.55)
+		)
+		(stroke
+			(width 0)
+			(type default)
+		)
+	)
 	(bus
 		(pts
@@
 		(pts
 			(xy 121.92 73.66) (xy 121.92 76.2)
+		)
+		(stroke
+			(width 0)
+			(type default)
+		)
+	)
+	(wire
+		(pts
+			(xy 219.71 74.93) (xy 223.52 74.93)
 		)
 		(stroke
@@
 		)
 	)
+	(label "GPIO8"
+		(at 223.52 77.47 0)
+		(effects
+			(font
+				(size 1.27 1.27)
+			)
+			(justify left bottom)
+		)
+	)
 	(label "GPIO22"
 		(at 125.73 101.6 0)
@@
 		)
 	)
+	(label "GPIO24"
+		(at 223.52 72.39 0)
+		(effects
+			(font
+				(size 1.27 1.27)
+			)
+			(justify left bottom)
+		)
+	)
 	(label "SD_CMD"
 		(at 124.46 73.66 0)
@@
 		)
 	)
+	(label "GPIO7"
+		(at 223.52 80.01 0)
+		(effects
+			(font
+				(size 1.27 1.27)
+			)
+			(justify left bottom)
+		)
+	)
 	(label "GPIO15"
 		(at 124.46 81.28 0)
@@
 		)
 	)
+	(label "GPIO23"
+		(at 223.52 69.85 0)
+		(effects
+			(font
+				(size 1.27 1.27)
+			)
+			(justify left bottom)
+		)
+	)
 	(label "SD_DAT3"
 		(at 124.46 66.04 0)
@@
 		)
 	)
+	(label "GPIO12"
+		(at 223.52 82.55 0)
+		(effects
+			(font
+				(size 1.27 1.27)
+			)
+			(justify left bottom)
+		)
+	)
 	(label "GPIO25"
 		(at 171.45 55.88 0)
@@
 		)
 	)
+	(label "GPIO18"
+		(at 223.52 85.09 0)
+		(effects
+			(font
+				(size 1.27 1.27)
+			)
+			(justify left bottom)
+		)
+	)
 	(label "GPIO12"
 		(at 180.34 81.28 180)
@@
 	(label "GPIO14"
 		(at 124.46 78.74 0)
+		(effects
+			(font
+				(size 1.27 1.27)
+			)
+			(justify left bottom)
+		)
+	)
+	(label "GPIO25"
+		(at 223.52 74.93 0)
 		(effects
 			(font
@@
 		)
 	)
+	(hierarchical_label "DEVSLP"
+		(shape input)
+		(at 219.71 69.85 180)
+		(effects
+			(font
+				(size 1.27 1.27)
+			)
+			(justify right)
+		)
+	)
 	(hierarchical_label "{SD}"
 		(shape bidirectional)
@@
 		)
 	)
+	(hierarchical_label "PEDET"
+		(shape output)
+		(at 218.44 82.55 180)
+		(effects
+			(font
+				(size 1.27 1.27)
+			)
+			(justify right)
+		)
+	)
+	(hierarchical_label "PEWAKE#"
+		(shape bidirectional)
+		(at 219.71 77.47 180)
+		(effects
+			(font
+				(size 1.27 1.27)
+			)
+			(justify right)
+		)
+	)
+	(hierarchical_label "PERST#"
+		(shape input)
+		(at 219.71 72.39 180)
+		(effects
+			(font
+				(size 1.27 1.27)
+			)
+			(justify right)
+		)
+	)
+	(hierarchical_label "LED1#"
+		(shape output)
+		(at 218.44 85.09 180)
+		(effects
+			(font
+				(size 1.27 1.27)
+			)
+			(justify right)
+		)
+	)
 	(hierarchical_label "{SD}"
 		(shape bidirectional)
@@
 		)
 	)
+	(hierarchical_label "CLKREQ#"
+		(shape bidirectional)
+		(at 219.71 74.93 180)
+		(effects
+			(font
+				(size 1.27 1.27)
+			)
+			(justify right)
+		)
+	)
+	(hierarchical_label "SUSCLK"
+		(shape input)
+		(at 218.44 80.01 180)
+		(effects
+			(font
+				(size 1.27 1.27)
+			)
+			(justify right)
+		)
+	)
 	(hierarchical_label "{GPIO}"
 		(shape bidirectional)
@@
 			)
 			(justify left)
-		)
-	)
-	(hierarchical_label "GPIO_VREF"
-		(shape output)
-		(at 57.15 72.39 0)
-		(effects
-			(font
-				(size 1.5 1.5)
-			)
-			(justify left)
