File: ulx5m-m2.kicad_pcb (KiCad board)
At the start: 6 copper layers, 110.1 x 106 mm, 323 parts, among them J1 DF40C-100DP-0.4V_51_, J2 DF40C-100DP-0.4V_51_, J3 Vcore_sel, J4 JTAG, J5 USB_C_Receptacle, Q1 BSS138, Q2 BSS138, SW1 219-2MST, U1 TLV62569DBV, U10 IS42S16320D-6BLI, U14 KSZ9031RNXCA, U2 TLV62569DBV, U3 MPM3833CGRH-Z, U4 GateMate-CCGM1A1, U5 TLV62569DBV, U6 74LVC1G04GM,115, U7 74LVC2G00HK3-7, U8 74LVC2G00HK3-7, U9 AT25QL321-MBUE-T, X1 ECS-2520MV-250-xx, X2 511FCA100M000BAG, Y1 ASE2-25.000MHZ-L-C-T

Commit message: cleanup
Parts:
- removed C134, C135: 100n, Capacitor_SMD:C_0402_1005Metric
- removed C3: 4u7, Capacitor_SMD:C_0402_1005Metric
- removed C59, C60, C61, C62, C63, C64, C65, C66: 220n, Capacitor_SMD:C_0402_1005Metric
- removed C7: 10u, Capacitor_SMD:C_0402_1005Metric
- removed C9: 1u, Capacitor_SMD:C_0402_1005Metric
- removed H1, H2, H3, H4: MountingHole, MountingHole:MountingHole_2.7mm_M2.5_DIN965_Pad
- removed J1, J2: DF40C-100DP-0.4V_51_, ulx5m-gs:HRS_DF40C-100DP-0.4V_51_
- removed J10: ~, PCIexpress:M.2 M Key Connector
- removed L2: DFE322512F-2R2M=P2, Inductor_SMD:L_1008_2520Metric
- removed R11: 0R, Resistor_SMD:R_0603_1608Metric
- removed R5: 100k, Resistor_SMD:R_0402_1005Metric
- removed R6: 22k, Resistor_SMD:R_0402_1005Metric
- removed TP2: 3V3, TestPoint:TestPoint_Pad_D1.0mm
- removed U2: TLV62569DBV, Package_TO_SOT_SMD:SOT-23-5
- moved R115 110.7 mm to (163.8, 126.8), turned to -90 degrees
- moved C141 110.7 mm to (165.1, 126.2), turned to 90 degrees
- moved SW1 110.7 mm to (168.4, 124.7), turned to -90 degrees
- moved C140 110.6 mm to (166.4, 125.6), turned to -90 degrees
- moved U6 110.6 mm to (171.7, 123.0), turned to 0 degrees
- moved R116 110.2 mm to (162.8, 126.8), turned to -90 degrees
- moved U7 108.5 mm to (171.8, 121.3), turned to 0 degrees
- moved C90 108.1 mm to (162.4, 125.4), turned to 180 degrees
- moved C88 107.2 mm to (164.3, 123.9), turned to 0 degrees
- moved C89 106.1 mm to (162.4, 123.9), turned to 180 degrees
- moved R35 106.1 mm to (172.9, 118.7), turned to 180 degrees
- moved C94 105.7 mm to (167.0, 121.5), turned to 180 degrees
- moved R36 105.5 mm to (171.7, 118.9), turned to -90 degrees
- moved R41 105.3 mm to (170.7, 119.3), turned to 90 degrees
- moved R43 104.7 mm to (169.7, 119.3), turned to 90 degrees
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Connections:
- net /PET1+ renamed /M.2 M Key/PETp1
- net /PET1- renamed /M.2 M Key/PETn1
- net /PET2+ renamed /M.2 M Key/PETp2
- net /PET2- renamed /M.2 M Key/PETn2
- net /PET3+ renamed /M.2 M Key/PETp3
- net /PET3- renamed /M.2 M Key/PETn3
- net /cm4-gpio/GPIO12 renamed /config/GPIO12
- net /cm4-gpio/GPIO16 renamed /config/GPIO16
- net /cm4-gpio/GPIO20 renamed /config/GPIO20
- net /cm4-gpio/GPIO21 renamed /config/GPIO21
- net /cm4-gpio/USB_CC1 renamed /ethernet/USB_CC1
- net /cm4-gpio/USB_CC2 renamed /ethernet/USB_CC2
- net /cm4-hsio/LVDS0_C_N renamed /lvds/LVDS0_C_N
- net /cm4-hsio/LVDS0_C_P renamed /lvds/LVDS0_C_P
- net /cm4-hsio/LVDS0_D0_N renamed /lvds/LVDS0_D0_N
- net /cm4-hsio/LVDS0_D0_P renamed /lvds/LVDS0_D0_P
- net /cm4-hsio/LVDS0_D1_N renamed /lvds/LVDS0_D1_N
- net /cm4-hsio/LVDS0_D1_P renamed /lvds/LVDS0_D1_P
- net /cm4-hsio/LVDS0_D2_N renamed /lvds/LVDS0_D2_N
- net /cm4-hsio/LVDS0_D2_P renamed /lvds/LVDS0_D2_P
- net /cm4-hsio/LVDS0_D3_N renamed /lvds/LVDS0_D3_N
- net /cm4-hsio/LVDS0_D3_P renamed /lvds/LVDS0_D3_P
- net /cm4-hsio/LVDS1_C_N renamed /lvds/LVDS1_C_N
- net /cm4-hsio/LVDS1_C_P renamed /lvds/LVDS1_C_P
- net /cm4-hsio/LVDS1_D0_N renamed /lvds/LVDS1_D0_N
- net /cm4-hsio/LVDS1_D0_P renamed /lvds/LVDS1_D0_P
- net /cm4-hsio/LVDS1_D1_N renamed /lvds/LVDS1_D1_N
- net /cm4-hsio/LVDS1_D1_P renamed /lvds/LVDS1_D1_P
- net /cm4-hsio/LVDS1_D2_N renamed /lvds/LVDS1_D2_N
- net /cm4-hsio/LVDS1_D2_P renamed /lvds/LVDS1_D2_P
- net /cm4-hsio/PCIe_RX_N renamed /M.2 M Key/PCIe_RX_N
- net /cm4-hsio/PCIe_RX_P renamed /M.2 M Key/PCIe_RX_P
- net /cm4-hsio/USB_N renamed /ethernet/USB_N
- net /cm4-hsio/USB_P renamed /ethernet/USB_P
- C136 pad 2: /cm4-hsio/PCIe_CLK_P -> /M.2 M Key/PCIe_CLK_P
- C137 pad 2: /cm4-hsio/PCIe_CLK_N -> /M.2 M Key/PCIe_CLK_N
- C143 pad 2: /PET0- -> /M.2 M Key/PCIe_TX_N
- C144 pad 2: /PET0+ -> /M.2 M Key/PCIe_TX_P
- Q1 pad 3: /cm4-gpio/ETH0_LEDY -> /ethernet/ETH0_LEDY
- Q2 pad 3: /cm4-gpio/ETH0_LEDG -> /ethernet/ETH0_LEDG
- R110 pad 1: /serdes/PCIe_TX_BC_P -> /M.2 M Key/PCIe_TX_P
- R110 pad 2: /serdes/PCIe_TX_BC_N -> /M.2 M Key/PCIe_TX_N
- R128 pad 2: Net-(J2-Pad73) -> unconnected-(R128-Pad2)
- R134 pad 2: Net-(J2-Pad75) -> unconnected-(R134-Pad2)
- R138 pad 2: Net-(J2-Pad97) -> unconnected-(R138-Pad2)
- R139 pad 1: Net-(J2-Pad100) -> unconnected-(R139-Pad1)
- U14 pad 10: /cm4-gpio/ETH3_P -> /ethernet/ETH3_P
- U14 pad 11: /cm4-gpio/ETH3_N -> /ethernet/ETH3_N
- U14 pad 2: /cm4-gpio/ETH0_P -> /ethernet/ETH0_P
- U14 pad 3: /cm4-gpio/ETH0_N -> /ethernet/ETH0_N
- U14 pad 5: /cm4-gpio/ETH1_P -> /ethernet/ETH1_P
- U14 pad 6: /cm4-gpio/ETH1_N -> /ethernet/ETH1_N
- U14 pad 7: /cm4-gpio/ETH2_P -> /ethernet/ETH2_P
- U14 pad 8: /cm4-gpio/ETH2_N -> /ethernet/ETH2_N
- U4 pad A11: /cm4-gpio/GPIO8 -> /config/GPIO8
- U4 pad A4: /cm4-gpio/SD_DAT0 -> /gpio/SD_DAT0
- U4 pad A6: /cm4-gpio/GPIO14 -> /config/GPIO14
- U4 pad A8: /cm4-gpio/GPIO18 -> /config/GPIO18
- U4 pad A9: /cm4-gpio/GPIO24 -> /config/GPIO24
- U4 pad B11: /cm4-gpio/GPIO7 -> /config/GPIO7
- U4 pad B5: /cm4-gpio/SD_DAT3 -> /gpio/SD_DAT3
- U4 pad B6: /cm4-gpio/GPIO15 -> /config/GPIO15
- U4 pad B8: /cm4-gpio/GPIO23 -> /config/GPIO23
- U4 pad B9: /cm4-gpio/GPIO25 -> /config/GPIO25
- U4 pad C10: /cm4-gpio/GPIO10 -> /config/GPIO10
- U4 pad C11: /cm4-gpio/GPIO11 -> /config/GPIO11
- U4 pad C12: /cm4-gpio/GPIO5 -> /config/GPIO5
- U4 pad C13: /cm4-gpio/GPIO6 -> /config/GPIO6
- U4 pad C14: /cm4-gpio/GPIO19 -> /config/GPIO19
- U4 pad C5: /cm4-gpio/SD_DAT2 -> /gpio/SD_DAT2
- U4 pad C6: /cm4-gpio/SD_CLK -> /gpio/SD_CLK
- U4 pad C7: /cm4-gpio/GPIO3 -> /config/GPIO3
- U4 pad C8: /cm4-gpio/GPIO17 -> /config/GPIO17
- U4 pad C9: /cm4-gpio/GPIO27 -> /config/GPIO27
- U4 pad D10: /cm4-gpio/GPIO9 -> /config/GPIO9
- U4 pad D11: /cm4-gpio/FAN_PWM -> /gpio/FAN_PWM
- U4 pad D12: /cm4-gpio/SD_DAT1 -> /gpio/SD_DAT1
- U4 pad D13: /cm4-gpio/GPIO13 -> /config/GPIO13
- U4 pad D14: /cm4-gpio/GPIO26 -> /config/GPIO26
- U4 pad D6: /cm4-gpio/SD_CMD -> /gpio/SD_CMD
- U4 pad D7: /cm4-gpio/GPIO2 -> /config/GPIO2
- U4 pad D8: /cm4-gpio/GPIO4 -> /config/GPIO4
- U4 pad D9: /cm4-gpio/GPIO22 -> /config/GPIO22
- U4 pad G16: unconnected-(U4D-IO_EA_A8-PadG16) -> /LED1#
- U4 pad G17: unconnected-(U4D-IO_EA_B7-PadG17) -> /PEDET
- U4 pad G18: PWR_BTN -> /SUSCLK
- U4 pad H15: /cm4-gpio/ID_SC -> /PEWAKE#
- U4 pad H16: /cm4-gpio/ID_SD -> /CLKREQ#
- U4 pad J15: /cm4-gpio/SCL0 -> /PERST#
- U4 pad J16: /cm4-gpio/SDA0 -> /DEVSLP
- U4 pad K16: /cm4-hsio/USB_OTG_ID -> /ethernet/USB_OTG_ID
- U4 pad U13: /serdes/PCIe_TX_BC_P -> /M.2 M Key/PCIe_TX_P
- U4 pad V13: /serdes/PCIe_TX_BC_N -> /M.2 M Key/PCIe_TX_N
Routing:
- net VDD_CLK: track 408.2 -> 156.3 mm, vias 52 -> 45
- net +3V3: track 271.2 -> 82.0 mm, vias 32 -> 26
- net +5V: track 138.2 -> 8.34 mm, vias 21 -> 11
- net SDRAM_VCC: track 345.0 -> 217.7 mm, vias 45 -> 37
- net +1V2: track 100.6 -> 18.6 mm
- net VDD_CORE: track 342.4 -> 261.3 mm
- net GND: track 1368.5 -> 1321.4 mm, vias 299 -> 211
- net PWR_BTN: track 42.2 -> 0.00 mm, vias 3 -> 0
- net RST_N: track 105.7 -> 70.1 mm, vias 8 -> 5
- net /cm4-gpio/SDA0: track 32.8 -> 0.00 mm, vias 2 -> 0
- net /cm4-hsio/USB_OTG_ID: track 32.5 -> 0.00 mm, vias 2 -> 0
- net /cm4-gpio/ETH0_P: track 31.6 -> 0.00 mm, vias 1 -> 0
- net /DEVSLP: track 0.00 -> 31.2 mm, vias 0 -> 2
- net /cm4-gpio/ID_SD: track 30.9 -> 0.00 mm, vias 2 -> 0
- net /cm4-gpio/ETH0_N: track 30.9 -> 0.00 mm, vias 1 -> 0
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- removed copper zone on In3.Cu, net +1V2
- removed copper zone on In3.Cu, net +3V3
- removed copper zone on In3.Cu, net +5V
- removed copper zone on In3.Cu, net /config/+1V8_FLASH
- removed copper zone on In3.Cu, net /lvds/+1V2_SA
- removed copper zone on In3.Cu, net /lvds/+1V8_SB
- removed copper zone on In1.Cu, net GND
- removed copper zone on In3.Cu, net GND
- removed copper zone on In4.Cu, net GND
- removed copper zone on In3.Cu, net SDRAM_VCC
- removed copper zone on In3.Cu, net VDD_CLK
- removed copper zone on In3.Cu, net VDD_CORE
- removed copper zone on In3.Cu, net VDD_SER
Other:
- board size 110.1 x 106 mm -> 30 x 106 mm
- board text removed: "3V3 1V8"
- board text removed: "5V"
- board text removed: "DDMI0"
- board text removed: "ETH"
- board text removed: "GPIO"
- board text removed: "I2C"
- board text removed: "SD"

Commit message: cleanup
Parts:
- removed R128, R134, R138, R139: 10k, Resistor_SMD:R_0402_1005Metric
- removed R129, R132, R135, R136: 150R, Resistor_SMD:R_0402_1005Metric
- added J10: ~, PCIexpress:M.2 M Key Connector, F.Cu at (158.3, 143.0)
- moved L1 53.2 mm to (155.8, 68.3), turned to -90 degrees
- moved C8 52.0 mm to (155.3, 70.8), turned to 0 degrees
- moved R10 51.9 mm to (155.6, 74.0), turned to 180 degrees
- moved C6 51.8 mm to (155.3, 71.8), turned to 0 degrees
- moved R4 49.1 mm to (153.4, 71.3), turned to 0 degrees
- moved U1 48.9 mm to (152.6, 68.2), turned to -90 degrees
- moved R3 48.5 mm to (153.1, 72.8), turned to 180 degrees
- moved C2 47.1 mm to (151.9, 71.3), turned to -90 degrees
- moved TP1 45.6 mm to (151.1, 73.3), turned to -90 degrees
Connections:
- net /M.2 M Key/PCIe_CLK_N renamed /serdes/PCIe_CLK_N
- net /M.2 M Key/PCIe_CLK_P renamed /serdes/PCIe_CLK_P
- net /M.2 M Key/PCIe_RX_N renamed /serdes/PCIe_RX_N
- net /M.2 M Key/PCIe_RX_P renamed /serdes/PCIe_RX_P
- net /config/GPIO10 renamed /gpio/GPIO10
- net /config/GPIO11 renamed /gpio/GPIO11
- net /config/GPIO13 renamed /gpio/GPIO13
- net /config/GPIO14 renamed /gpio/GPIO14
- net /config/GPIO15 renamed /gpio/GPIO15
- net /config/GPIO17 renamed /gpio/GPIO17
- net /config/GPIO18 renamed /gpio/GPIO18
- net /config/GPIO19 renamed /gpio/GPIO19
- net /config/GPIO2 renamed /gpio/GPIO2
- net /config/GPIO22 renamed /gpio/GPIO22
- net /config/GPIO23 renamed /gpio/GPIO23
- net /config/GPIO24 renamed /gpio/GPIO24
- net /config/GPIO25 renamed /gpio/GPIO25
- net /config/GPIO26 renamed /gpio/GPIO26
- net /config/GPIO27 renamed /gpio/GPIO27
- net /config/GPIO3 renamed /gpio/GPIO3
- net /config/GPIO4 renamed /gpio/GPIO4
- net /config/GPIO5 renamed /gpio/GPIO5
- net /config/GPIO6 renamed /gpio/GPIO6
- net /config/GPIO7 renamed /gpio/GPIO7
- net /config/GPIO8 renamed /gpio/GPIO8
- net /config/GPIO9 renamed /gpio/GPIO9
- R110 pad 1: /M.2 M Key/PCIe_TX_P -> /serdes/PCIe_TX_BC_P
- R110 pad 2: /M.2 M Key/PCIe_TX_N -> /serdes/PCIe_TX_BC_N
- U4 pad A12: /config/GPIO12 -> /gpio/GPIO12
- U4 pad A14: /config/GPIO20 -> /gpio/GPIO20
- U4 pad B12: /config/GPIO16 -> /gpio/GPIO16
- U4 pad B14: /config/GPIO21 -> /gpio/GPIO21
- U4 pad U13: /M.2 M Key/PCIe_TX_P -> /serdes/PCIe_TX_BC_P
- U4 pad V13: /M.2 M Key/PCIe_TX_N -> /serdes/PCIe_TX_BC_N
Routing:
- net RST_N: track 70.1 -> 39.8 mm
- net /lvds/LVDS1_D2_P: track 18.4 -> 0.00 mm, vias 1 -> 0
- net /lvds/LVDS1_D2_N: track 18.0 -> 0.00 mm, vias 1 -> 0
- net /lvds/LVDS1_C_P: track 15.0 -> 0.57 mm
- net /lvds/LVDS1_D1_N: track 15.0 -> 0.57 mm
- net /lvds/LVDS1_C_N: track 15.0 -> 0.57 mm
- net /lvds/LVDS1_D1_P: track 15.0 -> 0.57 mm
- net /M.2 M Key/PCIe_TX_P: track 12.2 -> 0.00 mm
- net /M.2 M Key/PCIe_TX_N: track 11.7 -> 0.00 mm
- net /lvds/LVDS0_D0_N: track 12.5 -> 1.02 mm
- net /serdes/PCIe_TX_BC_P: track 0.00 -> 11.3 mm
- net /lvds/LVDS1_D0_P: track 16.1 -> 5.02 mm
- net /lvds/LVDS1_D0_N: track 15.7 -> 4.73 mm
- net /serdes/PCIe_TX_BC_N: track 0.00 -> 10.8 mm
- net /lvds/LVDS0_D0_P: track 12.5 -> 2.36 mm
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- added copper zone on B.Cu, net (none)
- removed copper zone on B.Cu, net +3.3V
Other:
- board text removed: "DDMI0 - 28mm PCIe - 25mm LVDS0 - 14mm LVDS1 - 17mm"

Commit message: Version 1.0
Parts:
- removed C104, C105, C109, C114: 10u, Capacitor_SMD:C_0402_1005Metric
- removed C106, C107, C108, C112, C116, C117, C118: 100n, Capacitor_SMD:C_0402_1005Metric
- removed C110, C111, C113, C119: 10n, Capacitor_SMD:C_0402_1005Metric
- removed C115: 4u7, Capacitor_SMD:C_0402_1005Metric
- removed FB1, FB2, FB3: BLM18PG121SN1D, Inductor_SMD:L_0603_1608Metric
- removed Q1, Q2: BSS138, Package_TO_SOT_SMD:SOT-523
- removed R100, R101, R102, R104, R89, R90, R91, R92, R93, R94, R97, R98, R99: 27R, Resistor_SMD:R_0402_1005Metric
- removed R103: 12k1, Resistor_SMD:R_0402_1005Metric
- removed R130, R131, R50, R51, R54: 150R, Resistor_SMD:R_0402_1005Metric
- removed R147, R148, R149, R150: 10k, Resistor_SMD:R_0402_1005Metric
- removed R66, R67, R70, R71, R72, R73, R78, R79, R84, R85, R96: 4k7, Resistor_SMD:R_0402_1005Metric
- removed U14: KSZ9031RNXCA, Package_DFN_QFN:QFN-48-1EP_7x7mm_P0.5mm_EP5.15x5.15mm
- removed X1: ECS-2520MV-250-xx, Oscillator:Oscillator_SMD_ECS_2520MV-xxx-xx-4Pin_2.5x2.0mm
- removed kibuzzard-686AA8CB: G***, kibuzzard-686AA8CB
- removed kibuzzard-689F41CF: G***, kibuzzard-689F41CF
- removed kibuzzard-68DC261C: G***, kibuzzard-68DC261C
- added kibuzzard-6A16D9FF: G***, kibuzzard-6A16D9FF, F.Cu at (157.7, 41.9)
- C132, R58: moved to B.Cu
- R109, R27, R35, R38, R46, R61, R62: moved to F.Cu
- moved LoGo_opencologne 142.1 mm to (169.3, 69.7), turned to 90 degrees
- moved R29 141.8 mm to (169.5, 108.4), turned to 90 degrees
- moved D1 137.1 mm to (167.5, 123.0), turned to 0 degrees
- moved R31 136.1 mm to (167.5, 124.0), turned to 180 degrees
- moved G*** 134.9 mm to (147.0, 131.4)
- moved G*** 132.9 mm to (157.8, 39.8)
- moved U8 130.7 mm to (159.2, 130.5), turned to 90 degrees
- moved D5 127.5 mm to (170.1, 89.9), turned to -90 degrees
- moved C133 127.4 mm to (170.0, 94.7), turned to 0 degrees
- moved D6 126.5 mm to (171.5, 89.9), turned to 90 degrees
- moved R112 126.4 mm to (170.0, 95.8), turned to 180 degrees
- moved R113 126.3 mm to (168.1, 94.6), turned to 180 degrees
- moved R61 125.7 mm to (163.3, 63.2)
- moved R58 124.6 mm to (171.3, 79.0)
- moved radiona 124.4 mm to (151.0, 79.5), turned to 90 degrees
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Connections:
- C1 pad 1: +5V -> +3V3
- C11 pad 1: +5V -> +3V3
- C136 pad 2: /serdes/PCIe_CLK_P -> /M.2 M Key/PCIe_CLK_P
- C137 pad 2: /serdes/PCIe_CLK_N -> /M.2 M Key/PCIe_CLK_N
- C2 pad 1: +5V -> +3V3
- J10 pad 12: +3.3V -> +3V3
- J10 pad 14: +3.3V -> +3V3
- J10 pad 16: +3.3V -> +3V3
- J10 pad 18: +3.3V -> +3V3
- J10 pad 2: +3.3V -> +3V3
- J10 pad 4: +3.3V -> +3V3
- J10 pad 70: +3.3V -> +3V3
- J10 pad 72: +3.3V -> +3V3
- J10 pad 74: +3.3V -> +3V3
- R1 pad 1: +5V -> +3V3
- R107 pad 1: /serdes/PCIe_RX_P -> /M.2 M Key/PCIe_RX_P
- R107 pad 2: /serdes/PCIe_RX_N -> /M.2 M Key/PCIe_RX_N
- R110 pad 1: /serdes/PCIe_TX_BC_P -> /M.2 M Key/PCIe_TX_P
- R110 pad 2: /serdes/PCIe_TX_BC_N -> /M.2 M Key/PCIe_TX_N
- U1 pad 1: +5V -> +3V3
- U1 pad 4: +5V -> +3V3
- U3 pad 13: +5V -> +3V3
- U3 pad 14: +5V -> +3V3
- U4 pad A11: /gpio/GPIO8 -> /PEWAKE#
- U4 pad A12: /gpio/GPIO12 -> /PEDET
- U4 pad A15: /ethernet/RGMII_REFCLK -> unconnected-(U4D-IO_EB_B8-PadA15)
- U4 pad A17: /ethernet/RGMII_TX0 -> unconnected-(U4D-IO_EB_B5-PadA17)
- U4 pad A8: /gpio/GPIO18 -> /LED1#
- U4 pad A9: /gpio/GPIO24 -> /PERST#
- U4 pad B11: /gpio/GPIO7 -> /SUSCLK
- U4 pad B15: /ethernet/RGMII_RX_DV -> unconnected-(U4D-IO_EB_A8-PadB15)
- U4 pad B17: /ethernet/RGMII_TX1 -> unconnected-(U4D-IO_EB_A5-PadB17)
- U4 pad B8: /gpio/GPIO23 -> /DEVSLP
- U4 pad B9: /gpio/GPIO25 -> /CLKREQ#
- U4 pad C15: /ethernet/RGMII_INT_N -> unconnected-(U4D-IO_EB_B7-PadC15)
- U4 pad C16: /ethernet/RGMII_MDC -> unconnected-(U4D-IO_EB_B6-PadC16)
- U4 pad C17: /ethernet/RGMII_TX2 -> unconnected-(U4D-IO_EB_B4-PadC17)
- U4 pad C18: /ethernet/RGMII_TX3 -> unconnected-(U4D-IO_EB_A4-PadC18)
- U4 pad D15: /ethernet/RGMII_RX_CLK -> unconnected-(U4D-IO_EB_A7-PadD15)
- U4 pad D16: /ethernet/RGMII_MDIO -> unconnected-(U4D-IO_EB_A6-PadD16)
- U4 pad D17: /ethernet/RGMII_TX_CK -> unconnected-(U4D-IO_EB_B2-PadD17)
- U4 pad D18: /ethernet/RGMII_TXE -> unconnected-(U4D-IO_EB_A2-PadD18)
- U4 pad E15: /ethernet/RGMII_RST_N -> unconnected-(U4D-IO_EB_B3-PadE15)
- U4 pad E16: /ethernet/ETH_CLK -> unconnected-(U4D-IO_EB_A3-PadE16)
- U4 pad F15: /ethernet/RGMII_RXD3 -> unconnected-(U4D-IO_EB_B1-PadF15)
- U4 pad F16: /ethernet/RGMII_RXD2 -> unconnected-(U4D-IO_EB_A1-PadF16)
- U4 pad F17: /ethernet/RGMII_RXD1 -> unconnected-(U4D-IO_EB_B0-PadF17)
- U4 pad F18: /ethernet/RGMII_RXD0 -> unconnected-(U4D-IO_EB_A0-PadF18)
- U4 pad G16: /LED1# -> unconnected-(U4D-IO_EA_A8-PadG16)
- U4 pad G17: /PEDET -> unconnected-(U4D-IO_EA_B7-PadG17)
- U4 pad G18: /SUSCLK -> unconnected-(U4D-IO_EA_A7-PadG18)
- U4 pad H15: /PEWAKE# -> unconnected-(U4D-IO_EA_B6-PadH15)
- U4 pad H16: /CLKREQ# -> unconnected-(U4D-IO_EA_A6-PadH16)
- U4 pad J15: /PERST# -> unconnected-(U4D-IO_EA_B5-PadJ15)
- U4 pad J16: /DEVSLP -> unconnected-(U4D-IO_EA_A5-PadJ16)
- U4 pad U11: /serdes/PCIe_RX_P -> /M.2 M Key/PCIe_RX_P
- U4 pad U13: /serdes/PCIe_TX_BC_P -> /M.2 M Key/PCIe_TX_P
- U4 pad V11: /serdes/PCIe_RX_N -> /M.2 M Key/PCIe_RX_N
- U4 pad V13: /serdes/PCIe_TX_BC_N -> /M.2 M Key/PCIe_TX_N
- U5 pad 1: +5V -> +3V3
- U5 pad 4: +5V -> +3V3
Routing:
- net GND: track 1320.2 -> 833.8 mm, vias 213 -> 237
- net +3V3: track 77.8 -> 294.2 mm, vias 26 -> 29
- net VDD_CLK: track 156.3 -> 243.8 mm, vias 45 -> 29
- net RST_N: track 39.8 -> 105.4 mm, vias 5 -> 7
- net /M.2 M Key/PCIe_RX_P: track 0.00 -> 64.8 mm, vias 0 -> 2
- net /config/JTAG_TMS: track 72.6 -> 7.95 mm, vias 5 -> 0
- net /M.2 M Key/PCIe_RX_N: track 0.00 -> 63.4 mm, vias 0 -> 2
- net /M.2 M Key/PCIe_TX_P: track 0.00 -> 60.9 mm, vias 0 -> 2
- net /M.2 M Key/PCIe_TX_N: track 0.00 -> 60.0 mm, vias 0 -> 2
- net /LED1#: track 0.57 -> 53.8 mm
- net /config/JTAG_TDI: track 61.9 -> 11.1 mm, vias 4 -> 0
- net /PEDET: track 0.00 -> 48.4 mm, vias 0 -> 2
- net /serdes/SER_CLK_P: track 4.33 -> 52.1 mm, vias 0 -> 2
- net /serdes/SER_CLK_N: track 5.07 -> 52.1 mm, vias 0 -> 2
- net /config/JTAG_TCK: track 58.9 -> 13.1 mm, vias 4 -> 0
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- added copper zone on In1.Cu, net GND
- added copper zone on In2.Cu, net GND
- removed copper zone on B.Cu, net (none)
Other:
- copper layers 6 -> 4
- board text removed: "LVDS0"
- board text removed: "LVDS1"
- board text removed: "PCIe"
- board text removed: "TDI-GPIO12 TDO-GPIO16 TCK-GPIO20 TMS-GPIO21"
- board text removed: "USB"
