File: ulx5m-m2.kicad_pcb (KiCad board)
At the start: 4 copper layers, 30 x 106 mm, 231 parts, among them J3 Vcore_sel, J4 JTAG, J5 USB_C_Receptacle, SW1 219-2MST, U1 TLV62569DBV, U10 IS42S16320D-6BLI, U3 MPM3833CGRH-Z, U4 GateMate-CCGM1A1, U5 TLV62569DBV, U6 74LVC1G04GM,115, U7 74LVC2G00HK3-7, U8 74LVC2G00HK3-7, U9 AT25QL321-MBUE-T, X2 511FCA100M000BAG, Y1 ASE2-25.000MHZ-L-C-T

Commit message: Cleanup for v2 - we need to remove all modules, rotate FPGA, then assemble them together
Parts:
- JP1: moved to F.Cu
- moved J10 200.0 mm to (358.3, 143.0)
- moved R25 166.0 mm to (321.2, 138.7)
- moved R24 166.0 mm to (320.2, 138.7)
- moved SW1 166.0 mm to (321.2, 142.7)
- moved JP1 154.4 mm to (315.2, 146.4), turned to 180 degrees
- moved R29 148.1 mm to (314.0, 140.6)
- moved R30 148.1 mm to (311.9, 143.8)
- moved R27 148.1 mm to (313.1, 136.7)
- moved BTN2 121.0 mm to (47.7, 121.7)
- moved R118 121.0 mm to (44.1, 117.7)
- moved BTN1 121.0 mm to (46.1, 126.8)
- moved BTN3 121.0 mm to (46.8, 116.7)
- moved D10 121.0 mm to (53.1, 125.6)
- moved D11 121.0 mm to (53.1, 124.0)
- moved D12 121.0 mm to (53.1, 122.4)
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Routing:
- net +3V3: track 294.2 -> 141.9 mm, vias 29 -> 26
- net VDD_CLK: track 243.8 -> 127.8 mm, vias 29 -> 25
- net RST_N: track 105.4 -> 26.6 mm, vias 7 -> 5
- net /M.2 M Key/PCIe_RX_P: track 64.8 -> 6.44 mm, vias 2 -> 1
- net /M.2 M Key/PCIe_RX_N: track 63.4 -> 5.25 mm, vias 2 -> 1
- net /M.2 M Key/PCIe_TX_P: track 60.9 -> 5.25 mm, vias 2 -> 1
- net /M.2 M Key/PCIe_TX_N: track 60.0 -> 4.97 mm, vias 2 -> 1
- net /serdes/SER_CLK_P: track 52.1 -> 0.56 mm, vias 2 -> 1
- net /serdes/SER_CLK_N: track 52.1 -> 1.36 mm
- net /PEWAKE#: track 49.2 -> 0.57 mm, vias 1 -> 0
- net /SUSCLK: track 49.9 -> 1.77 mm, vias 1 -> 0
- net /LED1#: track 53.8 -> 5.90 mm
- net /PEDET: track 48.4 -> 0.66 mm, vias 2 -> 0
- net /CLKREQ#: track 48.8 -> 1.96 mm, vias 1 -> 0
- net /PERST#: track 47.5 -> 0.97 mm, vias 1 -> 0
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
Commit message: Chaning place of SDRAM
Parts:
- moved J10 200.0 mm to (158.3, 143.0)
- moved C4 44.7 mm to (171.1, 129.1), turned to 180 degrees
- moved R9 42.4 mm to (169.2, 129.1), turned to 0 degrees
- moved Y1 41.2 mm to (169.9, 126.3), turned to -90 degrees
- moved R122 40.9 mm to (168.2, 130.8), turned to 180 degrees
- moved TP6 40.7 mm to (168.2, 130.6), turned to 180 degrees
- moved R7 40.6 mm to (163.7, 133.8), turned to -90 degrees
- moved R8 40.4 mm to (164.7, 133.8), turned to -90 degrees
- moved C56 38.0 mm to (165.7, 130.6), turned to 180 degrees
- moved R23 37.9 mm to (166.7, 129.4), turned to 180 degrees
- moved C55 36.0 mm to (163.2, 130.9), turned to -90 degrees
- moved C54 35.0 mm to (162.2, 130.9), turned to -90 degrees
- moved C53 30.7 mm to (161.4, 127.5), turned to 180 degrees
- moved C38 29.7 mm to (161.4, 126.5), turned to 0 degrees
- moved R121 29.3 mm to (151.4, 132.1), turned to 180 degrees
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Connections:
- U4 pad A11: /PEWAKE# -> SDRAM_D13
- U4 pad A12: /PEDET -> SDRAM_D9
- U4 pad A14: /gpio/GPIO20 -> SDRAM_A5
- U4 pad A3: SDRAM_A1 -> SDRAM_nCS
- U4 pad A4: /gpio/SD_DAT0 -> SDRAM_A3
- U4 pad A6: /gpio/GPIO14 -> SDRAM_D2
- U4 pad A8: /LED1# -> SDRAM_BA0
- U4 pad A9: /PERST# -> SDRAM_A9
- U4 pad B11: /SUSCLK -> SDRAM_D14
- U4 pad B12: /gpio/GPIO16 -> SDRAM_D11
- U4 pad B14: /gpio/GPIO21 -> SDRAM_A8
- U4 pad B3: SDRAM_A2 -> SDRAM_nWE
- U4 pad B4: SDRAM_A10 -> SDRAM_D6
- U4 pad B5: /gpio/SD_DAT3 -> SDRAM_D3
- U4 pad B6: /gpio/GPIO15 -> SDRAM_D0
- U4 pad B8: /DEVSLP -> SDRAM_A6
- U4 pad B9: /CLKREQ# -> SDRAM_A11
- U4 pad C10: /gpio/GPIO10 -> SDRAM_CKE
- U4 pad C11: /gpio/GPIO11 -> SDRAM_D12
- U4 pad C12: /gpio/GPIO5 -> SDRAM_DQM1
- U4 pad C13: /gpio/GPIO6 -> SDRAM_A7
- U4 pad C14: /gpio/GPIO19 -> SDRAM_A4
- U4 pad C5: /gpio/SD_DAT2 -> SDRAM_D1
- U4 pad C6: /gpio/SD_CLK -> SDRAM_DQM0
- U4 pad C7: /gpio/GPIO3 -> SDRAM_D4
- U4 pad C8: /gpio/GPIO17 -> SDRAM_nRAS
- U4 pad C9: /gpio/GPIO27 -> SDRAM_BA1
- U4 pad D10: /gpio/GPIO9 -> SDRAM_CLK
- U4 pad D11: /gpio/FAN_PWM -> SDRAM_D15
- U4 pad D12: /gpio/SD_DAT1 -> SDRAM_D10
- U4 pad D13: /gpio/GPIO13 -> SDRAM_D8
- U4 pad D14: /gpio/GPIO26 -> SDRAM_A12
- U4 pad D6: /gpio/SD_CMD -> SDRAM_D7
- U4 pad D7: /gpio/GPIO2 -> SDRAM_D5
- U4 pad D8: /gpio/GPIO4 -> SDRAM_nCAS
- U4 pad D9: /gpio/GPIO22 -> SDRAM_A0
Routing:
- net VDD_CLK: track 127.8 -> 61.4 mm, vias 25 -> 8
- net VDD_CORE: track 280.0 -> 246.6 mm, vias 39 -> 34
- net SDRAM_A10: track 34.4 -> 2.89 mm
- net SDRAM_A1: track 31.3 -> 3.29 mm
- net SDRAM_A2: track 29.8 -> 2.36 mm
- net /config/SPI_CSN: track 27.9 -> 0.57 mm, vias 2 -> 1
- net GND: track 822.8 -> 799.7 mm, vias 206 -> 172
- net /ethernet/USB_PULL_N: track 25.7 -> 2.88 mm, vias 2 -> 0
- net SDRAM_A3: track 25.0 -> 6.04 mm, vias 2 -> 1
- net RST_N: track 26.6 -> 7.67 mm, vias 5 -> 3
- net SDRAM_A5: track 24.9 -> 6.83 mm, vias 2 -> 1
- net SDRAM_A4: track 22.0 -> 4.71 mm, vias 0 -> 1
- net SDRAM_A8: track 22.5 -> 6.39 mm
- net /ethernet/USB_PULL_P: track 17.0 -> 1.52 mm, vias 2 -> 0
- net /config/SPI_IO3: track 16.3 -> 1.50 mm, vias 1 -> 0
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
Commit message: update
Parts:
- removed C129, C130: 100n, Capacitor_SMD:C_0402_1005Metric
- C143, C144, C145, C146, C147, C148, C149, C150: footprint Capacitor_SMD:C_0201_0603Metric -> Capacitor_SMD:C_0402_1005Metric
- R144, R145, R146, R37: moved to F.Cu
- R34, R36, R39, R40, R41, R42, R43, X2: moved to B.Cu
- moved R33 137.7 mm to (127.6, 120.8)
- moved C48 137.7 mm to (127.7, 119.6)
- moved R35 137.7 mm to (132.9, 119.8)
- moved R38 137.7 mm to (133.9, 119.5)
- moved R37 124.4 mm to (139.7, 130.2), turned to 180 degrees
- moved BTN3 122.8 mm to (167.4, 93.6), turned to -90 degrees
- moved R146 122.4 mm to (167.5, 89.2), turned to 180 degrees
- moved R95 122.2 mm to (171.5, 98.2), turned to 90 degrees
- moved R88 120.9 mm to (169.9, 98.2), turned to 90 degrees
- moved U9 120.4 mm to (147.4, 127.4), turned to 0 degrees
- moved R87 119.6 mm to (168.3, 98.2), turned to 90 degrees
- moved D16 119.4 mm to (171.5, 100.7), turned to -90 degrees
- moved R86 118.3 mm to (166.7, 98.2), turned to 90 degrees
- moved D15 118.0 mm to (169.9, 100.7), turned to -90 degrees
- moved R65 117.1 mm to (165.1, 98.2), turned to 90 degrees
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Connections:
- net /lvds/ALED0 renamed /ethernet/ALED0
- net /lvds/ALED1 renamed /ethernet/ALED1
- net /lvds/ALED2 renamed /ethernet/ALED2
- net /lvds/ALED3 renamed /ethernet/ALED3
- net /lvds/ALED4 renamed /ethernet/ALED4
- net /lvds/ALED5 renamed /ethernet/ALED5
- net /lvds/ALED6 renamed /ethernet/ALED6
- net /lvds/ALED7 renamed /ethernet/ALED7
- C100 pad 1: VDD_CLK -> +3V3
- C102 pad 1: VDD_CLK -> +3V3
- C103 pad 1: VDD_CLK -> +3V3
- C136 pad 1: /serdes/SER_CLK_P -> /serdes/SER_CK_P
- C137 pad 1: /serdes/SER_CLK_N -> /serdes/SER_CK_N
- C98 pad 1: VDD_CLK -> +3V3
- D10 pad 2: /lvds/LED1 -> /ethernet/LED1
- D11 pad 2: /lvds/LED2 -> /ethernet/LED2
- D12 pad 2: /lvds/LED3 -> /ethernet/LED3
- D13 pad 2: /lvds/LED4 -> /ethernet/LED4
- D14 pad 2: /lvds/LED5 -> /ethernet/LED5
- D15 pad 2: /lvds/LED6 -> /ethernet/LED6
- D16 pad 2: /lvds/LED7 -> /ethernet/LED7
- D9 pad 2: /lvds/LED0 -> /ethernet/LED0
- U4 pad A11: SDRAM_D13 -> SDRAM_DQM0
- U4 pad A12: SDRAM_D9 -> SDRAM_D6
- U4 pad A14: SDRAM_A5 -> unconnected-(U4C-IO_NB_B7-PadA14)
- U4 pad A15: unconnected-(U4D-IO_EB_B8-PadA15) -> /ethernet/BTN2
- U4 pad A16: VDD_CLK -> +3V3
- U4 pad A17: unconnected-(U4D-IO_EB_B5-PadA17) -> /ethernet/LED3
- U4 pad A3: SDRAM_nCS -> SDRAM_D9
- U4 pad A4: SDRAM_A3 -> SDRAM_DQM1
- U4 pad A6: SDRAM_D2 -> SDRAM_A6
- U4 pad A8: SDRAM_BA0 -> SDRAM_nRAS
- U4 pad A9: SDRAM_A9 -> SDRAM_A3
- U4 pad B1: SDRAM_A12 -> SDRAM_D14
- U4 pad B11: SDRAM_D14 -> SDRAM_D5
- U4 pad B12: SDRAM_D11 -> SDRAM_D3
- U4 pad B14: SDRAM_A8 -> unconnected-(U4C-IO_NB_A7-PadB14)
- U4 pad B15: unconnected-(U4D-IO_EB_A8-PadB15) -> /ethernet/BTN3
- U4 pad B17: unconnected-(U4D-IO_EB_A5-PadB17) -> /ethernet/LED4
- U4 pad B18: VDD_CLK -> +3V3
- U4 pad B2: SDRAM_A4 -> SDRAM_D13
- U4 pad B3: SDRAM_nWE -> SDRAM_D10
- U4 pad B4: SDRAM_D6 -> SDRAM_D8
- U4 pad B5: SDRAM_D3 -> SDRAM_A12
- U4 pad B6: SDRAM_D0 -> SDRAM_A11
- U4 pad B8: SDRAM_A6 -> SDRAM_BA0
- U4 pad B9: SDRAM_A11 -> SDRAM_A10
- U4 pad C10: SDRAM_CKE -> SDRAM_A2
- U4 pad C11: SDRAM_D12 -> SDRAM_nCS
- U4 pad C12: SDRAM_DQM1 -> SDRAM_D7
- U4 pad C13: SDRAM_A7 -> SDRAM_D1
- U4 pad C14: SDRAM_A4 -> SDRAM_D0
- U4 pad C15: unconnected-(U4D-IO_EB_B7-PadC15) -> /ethernet/BTN1
- U4 pad C16: unconnected-(U4D-IO_EB_B6-PadC16) -> /ethernet/LED1
- U4 pad C17: unconnected-(U4D-IO_EB_B4-PadC17) -> /ethernet/LED5
- U4 pad C18: unconnected-(U4D-IO_EB_A4-PadC18) -> /ethernet/LED6
- U4 pad C3: SDRAM_A8 -> SDRAM_D11
- U4 pad C4: SDRAM_A5 -> SDRAM_D12
- U4 pad C5: SDRAM_D1 -> SDRAM_A8
- U4 pad C6: SDRAM_DQM0 -> SDRAM_A4
- U4 pad C7: SDRAM_D4 -> SDRAM_A9
- U4 pad C8: SDRAM_nRAS -> SDRAM_CKE
- U4 pad D1: SDRAM_D10 -> unconnected-(U4F-IO_WC_A5-PadD1)
- U4 pad D10: SDRAM_CLK -> SDRAM_A0
- U4 pad D11: SDRAM_D15 -> SDRAM_A1
- U4 pad D12: SDRAM_D10 -> SDRAM_nWE
- U4 pad D13: SDRAM_D8 -> SDRAM_D4
- U4 pad D14: SDRAM_A12 -> SDRAM_D2
- U4 pad D15: unconnected-(U4D-IO_EB_A7-PadD15) -> /ethernet/LED0
- U4 pad D16: unconnected-(U4D-IO_EB_A6-PadD16) -> /ethernet/LED2
- U4 pad D17: unconnected-(U4D-IO_EB_B2-PadD17) -> /ethernet/SD_CLK
- U4 pad D18: unconnected-(U4D-IO_EB_A2-PadD18) -> /ethernet/SD_CMD
- U4 pad D2: SDRAM_DQM1 -> unconnected-(U4F-IO_WC_B5-PadD2)
- U4 pad D3: SDRAM_D8 -> unconnected-(U4F-IO_WC_A6-PadD3)
- U4 pad D4: SDRAM_A7 -> SDRAM_D15
- U4 pad D6: SDRAM_D7 -> SDRAM_A5
- U4 pad D7: SDRAM_D5 -> SDRAM_A7
- U4 pad D8: SDRAM_nCAS -> SDRAM_CLK
- U4 pad D9: SDRAM_A0 -> SDRAM_nCAS
- U4 pad E1: SDRAM_D15 -> unconnected-(U4F-IO_WC_A3-PadE1)
- U4 pad E14: VDD_CLK -> +3V3
- U4 pad E15: unconnected-(U4D-IO_EB_B3-PadE15) -> /ethernet/LED7
- U4 pad E17: VDD_CLK -> +3V3
- U4 pad E2: SDRAM_D12 -> unconnected-(U4F-IO_WC_B3-PadE2)
- U4 pad E3: SDRAM_D11 -> unconnected-(U4F-IO_WC_A4-PadE3)
- U4 pad E4: SDRAM_D9 -> unconnected-(U4F-IO_WC_B4-PadE4)
- U4 pad F13: VDD_CLK -> +3V3
- U4 pad F15: unconnected-(U4D-IO_EB_B1-PadF15) -> /ethernet/SD_DAT3
- U4 pad F16: unconnected-(U4D-IO_EB_A1-PadF16) -> /ethernet/SD_DAT2
- U4 pad F17: unconnected-(U4D-IO_EB_B0-PadF17) -> /ethernet/SD_DAT1
- U4 pad F18: unconnected-(U4D-IO_EB_A0-PadF18) -> /ethernet/SD_DAT0
- U4 pad F3: SDRAM_D14 -> unconnected-(U4F-IO_WC_A2-PadF3)
- U4 pad F4: SDRAM_D13 -> unconnected-(U4F-IO_WC_B2-PadF4)
- U4 pad G1: SDRAM_A11 -> unconnected-(U4F-IO_WC_A0-PadG1)
- U4 pad G2: SDRAM_A9 -> unconnected-(U4F-IO_WC_B0-PadG2)
- U4 pad G3: SDRAM_CLK -> unconnected-(U4F-IO_WC_A1-PadG3)
- U4 pad G4: SDRAM_CKE -> unconnected-(U4F-IO_WC_B1-PadG4)
- U4 pad H1: SDRAM_BA0 -> unconnected-(U4F-IO_WB_A7-PadH1)
- U4 pad H2: SDRAM_A6 -> unconnected-(U4F-IO_WB_B7-PadH2)
- U4 pad H3: SDRAM_BA1 -> unconnected-(U4F-IO_WB_A8-PadH3)
- U4 pad H4: SDRAM_A0 -> unconnected-(U4F-IO_WB_B8-PadH4)
- U4 pad J17: /ethernet/BTN1 -> unconnected-(U4D-IO_EA_B4-PadJ17)
- U4 pad J18: /ethernet/BTN2 -> unconnected-(U4D-IO_EA_A4-PadJ18)
- U4 pad J3: SDRAM_nRAS -> unconnected-(U4F-IO_WB_A6-PadJ3)
- U4 pad J4: SDRAM_nCAS -> unconnected-(U4F-IO_WB_B6-PadJ4)
- U4 pad K1: SDRAM_D4 -> unconnected-(U4F-IO_WB_A5-PadK1)
- U4 pad K15: /ethernet/BTN3 -> unconnected-(U4D-IO_EA_B3-PadK15)
- U4 pad K2: SDRAM_D5 -> unconnected-(U4F-IO_WB_B5-PadK2)
- U4 pad K3: SDRAM_D2 -> unconnected-(U4F-IO_WB_A4-PadK3)
- U4 pad K4: SDRAM_D0 -> unconnected-(U4F-IO_WB_B4-PadK4)
- U4 pad L1: SDRAM_DQM0 -> unconnected-(U4F-IO_WB_A3-PadL1)
- U4 pad L2: SDRAM_D7 -> unconnected-(U4F-IO_WB_B3-PadL2)
- U4 pad L3: SDRAM_D3 -> unconnected-(U4F-IO_WB_A2-PadL3)
- U4 pad L4: SDRAM_D1 -> unconnected-(U4F-IO_WB_B2-PadL4)
- U4 pad M17: /lvds/LED7 -> /lvds/PEDET
- U4 pad M18: /lvds/LED6 -> /lvds/LED1#
- U4 pad M3: SDRAM_A3 -> unconnected-(U4F-IO_WB_A1-PadM3)
- U4 pad M4: SDRAM_D6 -> unconnected-(U4F-IO_WB_B1-PadM4)
- U4 pad N1: SDRAM_nCS -> unconnected-(U4F-IO_WB_A0-PadN1)
- U4 pad N2: SDRAM_nWE -> unconnected-(U4F-IO_WB_B0-PadN2)
- U4 pad P17: /lvds/LED5 -> /lvds/PEWAKE#
- U4 pad P18: /lvds/LED4 -> /lvds/SUSCLK
- U4 pad R17: /lvds/LED2 -> /lvds/PERST#
- U4 pad R18: /lvds/LED3 -> /lvds/CLKREQ#
- U4 pad U17: /lvds/LED0 -> unconnected-(U4E-IO_SB_A0-PadU17)
- U4 pad U18: /lvds/LED1 -> /lvds/DEVSLP
- X2 pad 4: /serdes/SER_CLK_P -> /serdes/SER_CK_P
- X2 pad 5: /serdes/SER_CLK_N -> /serdes/SER_CK_N
Routing:
- net VDD_CLK: track 61.4 -> 10.2 mm, vias 8 -> 2
- net +3V3: track 129.0 -> 170.3 mm, vias 23 -> 27
- net /ethernet/BTN1: track 4.31 -> 38.1 mm
- net /ethernet/BTN3: track 5.31 -> 38.5 mm, vias 1 -> 2
- net Net-(BTN1-Pad1): track 0.00 -> 30.9 mm
- net /ethernet/BTN2: track 2.65 -> 30.8 mm, vias 0 -> 2
- net /ethernet/LED7: track 0.00 -> 23.5 mm, vias 0 -> 2
- net /ethernet/LED0: track 0.00 -> 21.4 mm, vias 0 -> 2
- net /ethernet/LED2: track 0.00 -> 20.3 mm, vias 0 -> 2
- net /ethernet/LED1: track 0.00 -> 20.1 mm, vias 0 -> 2
- net /ethernet/LED6: track 0.00 -> 19.7 mm
- net /ethernet/LED5: track 0.00 -> 19.5 mm
- net /ethernet/LED4: track 0.00 -> 17.7 mm
- net /ethernet/LED3: track 0.00 -> 16.9 mm
- net /serdes/SER_CK_P: track 2.56 -> 16.1 mm, vias 1 -> 2
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