File: ulx5m-m2.kicad_sch (KiCad schematic)
At the start: 4 parts

Commit message: cleanup
Parts:
- removed H1, H2, H3, H4: MountingHole, MountingHole:MountingHole_2.7mm_M2.5_DIN965_Pad, symbol Mechanical:MountingHole_Pad
Connections:
- no-connect marks 7 -> 0
Other:
- removed sheet cm4-gpio
- removed sheet cm4-hsio
- sheet M.2 M Key ports: added {PCIe}; removed PERn0, PERn1, PERn2, PERn3, PERp0, PERp1, PERp2, PERp3, PETn0, PETn1, PETn2, PETn3, PETp0, PETp1, PETp2, PETp3, REFCLKn, REFCLKp
- sheet ethernet ports: added CLKREQ#, DEVSLP, LED1#, PEDET, PERST#, PEWAKE#, SUSCLK; removed none

Commit message: Version 1.0
Other:
- sheet ethernet ports: added none; removed CLKREQ#, DEVSLP, LED1#, PEDET, PERST#, PEWAKE#, SUSCLK
- sheet gpio ports: added CLKREQ#, DEVSLP, LED1#, PEDET, PERST#, PEWAKE#, SUSCLK; removed none
- note added: "Add RP2040 so that we do not need externa JTAG"
