File: ulx5m-m2.kicad_sch (KiCad schematic)
At the start: 0 parts

Commit message: Switching to 6L board - routing - adding schemaitcs
Parts:
- added FID101, FID102, FID103, FID104, FID105, FID106: Fiducial, Fiducial:Fiducial_0.75mm_Mask1.5mm, symbol Mechanical:Fiducial
